File: Flatline.kicad_sch (KiCad schematic)
At the start: 45 parts, among them J1 IN/LED/GND/OUT, J2 9V, J3 GND, J4 IN GND, J5 OUT GND, SW1 RELEASE, U1 OPA2134, U2 TL072, U3 Vactrol

Commit message: Flatline+: TIGHT side-chain high-pass switch (C14 100n + SW2), ON LED moved to the top row, re-routed; 1590B drill guide
Co-Authored-By: Claude Opus 5.5 <noreply@anthropic.com>
Parts:
- added C14: 100n, Capacitor_SMD:C_0805_2012Metric_Pad1.18x1.45mm_HandSolder, symbol Device:C
- added SW2: TIGHT, Flatline:SW_Taiway_200_SPDT, symbol Switch:SW_SPDT
Connections:
- net WET: now also C14.1, SW2.2 (B); no longer R8.1
- new net: C14.2, R8.1, SW2.1 (A)
- no-connect marks 1 -> 2
Other:
- note added: "1x4 ribbon to the footswitch board. \nIN GND / OUT GND: jack sleeves (star ground)."
- note added: "TIGHT (v1.1): C14 in series with R8. SW2 closed = C14 shorted (off)."
- note removed: "1x4 ribbon to the footswitch board. IN GND / OUT GND: jack sleeves (star ground)."
- moved on the sheet: C12, C13, C6, C7, C8, C9, D2, D3, D4, D5, D6, D7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
