File: Flatline.kicad_pcb (KiCad board)
At the start: 2 copper layers, 45 x 50 mm, 46 parts, among them J1 IN/LED/GND/OUT, J2 9V, J3 GND, J4 IN GND, J5 OUT GND, SW1 RELEASE, U1 OPA2134, U2 TL072, U3 Vactrol

Commit message: Flatline+: TIGHT side-chain high-pass switch (C14 100n + SW2), ON LED moved to the top row, re-routed; 1590B drill guide
Co-Authored-By: Claude Opus 5.5 <noreply@anthropic.com>
Parts:
- added C14: 100n, Capacitor_SMD:C_0805_2012Metric_Pad1.18x1.45mm_HandSolder, F.Cu at (46.5, 45.5)
- added SW2: TIGHT, Flatline:SW_Taiway_200_SPDT, B.Cu at (60.0, 51.5)
- moved D7 24.5 mm to (47.8, 31.0)
- moved D6 3.00 mm to (41.8, 31.0)
- moved C1 0.25 mm to (49.5, 27.2)
- moved C3 0.25 mm to (58.5, 46.2), turned to 180 degrees
- turned R15 to 180 degrees
Connections:
- R8 pad 1: /WET -> Net-(SW2-A)
Routing:
- net Net-(D7-A): track 5.03 -> 36.3 mm, vias 0 -> 1
- net /LED_K: track 33.4 -> 59.0 mm
- net GND: track 175.1 -> 150.4 mm, vias 1 -> 2
- net Net-(U1A-+): track 17.1 -> 38.5 mm
- net Net-(RV3-Pad2): track 42.7 -> 23.9 mm
- net /BR_N: track 112.2 -> 95.7 mm, vias 1 -> 0
- net Net-(SW2-A): track 0.00 -> 15.7 mm, vias 0 -> 1
- net /SC_N: track 44.8 -> 29.4 mm, vias 0 -> 2
- net /VB: track 102.9 -> 91.0 mm, vias 1 -> 2
- net Net-(U2B--): track 33.9 -> 23.7 mm
- net /SC_P: track 45.0 -> 35.3 mm, vias 2 -> 0
- net Net-(R6-Pad2): track 27.9 -> 20.3 mm
- net /OUT: track 35.5 -> 42.6 mm, vias 1 -> 2
- net Net-(SW1-A): track 37.8 -> 44.9 mm
- net /BR_P: track 45.5 -> 39.0 mm
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
Commit message: Flatline+: board name text (Flatline+ V1.0 / Super-Freq.com), zones refilled; ready for fab
Co-Authored-By: Claude Opus 5.5 <noreply@anthropic.com>
Other:
- board text added: "Flatline+ V1.0"
- board text added: "Super-Freq.com"
Changed lines of the file:
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@@
 		(layer "Edge.Cuts")
+	)
+	(gr_text "Super-Freq.com"
+		(at 43.2 42.55 0)
+		(layer "F.SilkS")
+		(effects
+			(font
+				(size 0.8 0.8)
+				(thickness 0.16)
+			)
+		)
+	)
+	(gr_text "Flatline+ V1.0"
+		(at 43.2 40.65 0)
+		(layer "F.SilkS")
+		(effects
+			(font
+				(size 1 1)
+				(thickness 0.16)
+			)
+		)
 	)
 	(segment
